File: BRD/gatilhov1.brd (EAGLE design)
At the start: 41.3 x 21.6 mm, 38 parts, among them IC1 TINY13-20SSU, IC2 LD117AS28TR, Q1 IRL7843, T1 BC817, T2 BC807, T3 BC817

Commit message: Signed-off-by: Jéfferson Pimenta Melo <jefferson.pimenta@hotmail.com>
Parts:
- removed C1: 100nF, rcl:C0805K
- removed C5: 10nF, rcl:C0805K
- added C4: 100nF, rcl:C1206K
- moved D5 11.0 mm to (9.67, 19.2), turned to 0 degrees
- moved SJ3 4.50 mm to (39.1, 10.7)
- moved R2 2.80 mm to (8.26, 7.36)
- moved T1 2.11 mm to (10.3, 10.6)
- moved T2 1.81 mm to (5.28, 10.6)
- moved M- 1.80 mm to (15.8, 19.4)
- moved R13 0.51 mm to (9.43, 17.6)
- moved R10 0.50 mm to (6.99, 17.6)
- moved R12 0.50 mm to (4.13, 17.6)
- moved T3 0.30 mm to (15.6, 17.4)
- moved R7 0.10 mm to (29.9, 12.1)
Connections:
- removed net N$3: C2.2, IC1.8, IC2.4, R5.2, R6.2, R7.2
- new net N$20: C2.2, C4.2, IC1.8, IC2.4, R10.1, R5.2, R6.2, R7.2, T2.E
- net N$1: now also C4.1; no longer C5.1, D5.A
- net N$14: now also D5.C; no longer C1.2, R10.1, T2.E
- net N$2: now also D5.A; no longer C1.1, D5.C
- net N$5: no longer C5.2
Routing:
- net N$20: track 0.00 -> 29.0 mm, vias 0 -> 2
- net N$3: track 22.1 -> 0.00 mm, vias 1 -> 0
- net N$14: track 31.3 -> 23.5 mm, vias 3 -> 2
- net N$2: track 20.4 -> 26.6 mm
- net N$19: track 12.3 -> 7.79 mm
- net N$17: track 7.63 -> 4.83 mm
- net N$15: track 2.71 -> 5.10 mm
- net N$16: track 3.11 -> 5.03 mm

Commit message: Signed-off-by: Jéfferson Pimenta Melo <jefferson.pimenta@hotmail.com>
Parts:
- added R14: 10k, resistor:R0805
- moved R1 0.10 mm to (16.5, 12.9)
Connections:
- net N$1: now also R14.1
- net N$6: now also R14.2
Routing:
- net N$6: track 10.9 -> 11.8 mm
Changed lines of the file:
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@@
 <attribute name="VALUE" x="18.57" y="19.467503125" size="0.0254" layer="27" rot="R270"/>
 </element>
-<element name="R1" library="resistor" package="R0805" value="1k" x="16.51" y="13.017503125" smashed="yes" rot="MR90">
-<attribute name="NAME" x="13.97" y="13.017503125" size="1.27" layer="26" rot="MR90"/>
-<attribute name="VALUE" x="13.97" y="12.382503125" size="1.27" layer="28" rot="MR90"/>
+<element name="R1" library="resistor" package="R0805" value="1k" x="16.51" y="12.917503125" smashed="yes" rot="MR90">
+<attribute name="NAME" x="13.97" y="12.917503125" size="1.27" layer="26" rot="MR90"/>
+<attribute name="VALUE" x="13.97" y="12.282503125" size="1.27" layer="28" rot="MR90"/>
 </element>
 <element name="R5" library="resistor" package="R0805" value="10k" x="26.67" y="7.302503125" smashed="yes" rot="MR0">
@@
 </element>
 <element name="C4" library="rcl" package="C1206K" value="100nF" x="9.4" y="14.2" rot="MR0"/>
+<element name="R14" library="resistor" package="R0805" value="10k" x="16.5" y="9.4" rot="MR90"/>
 </elements>
 <signals>
@@
 <wire x1="12.192" y1="7.366" x2="12.192" y2="7.112" width="0.4064" layer="1"/>
 <contactref element="C4" pad="1"/>
+<contactref element="R14" pad="1"/>
 <wire x1="12.065" y1="7.302503125" x2="12.192" y2="7.366" width="0" layer="19" extent="1-1"/>
 <wire x1="24.335" y1="2.857503125" x2="17.78" y2="4.762503125" width="0" layer="19" extent="16-16"/>
@@
 <via x="35.8775" y="11.112503125" extent="1-16" drill="1" shape="square"/>
 <via x="14.9225" y="11.112503125" extent="1-16" drill="1" shape="square"/>
-<wire x1="16.51" y1="12.067503125" x2="15.2425" y2="12.067503125" width="0.4064" layer="16"/>
-<wire x1="15.2425" y1="12.067503125" x2="14.9225" y2="11.747503125" width="0.4064" layer="16"/>
-<wire x1="14.9225" y1="11.747503125" x2="14.9225" y2="11.112503125" width="0.4064" layer="16"/>
 <wire x1="31.229" y1="6.667503125" x2="34.967503125" y2="6.667503125" width="0.4064" layer="1"/>
 <wire x1="34.967503125" y1="6.667503125" x2="35.9" y2="7.6" width="0.4064" layer="1"/>
 <wire x1="35.9" y1="7.6" x2="35.9" y2="11.090003125" width="0.4064" layer="1"/>
 <wire x1="35.9" y1="11.090003125" x2="35.8775" y2="11.112503125" width="0.4064" layer="1"/>
-<wire x1="16.51" y1="12.067503125" x2="31.229" y2="6.667503125" width="0" layer="19" extent="1-16"/>
+<contactref element="R14" pad="2"/>
+<wire x1="16.51" y1="11.967503125" x2="16.51" y2="11.1" width="0.4064" layer="16"/>
+<wire x1="16.51" y1="11.1" x2="16.51" y2="10.36" width="0.4064" layer="16"/>
+<wire x1="16.51" y1="10.36" x2="16.5" y2="10.35" width="0.4064" layer="16"/>
+<wire x1="14.9225" y1="11.112503125" x2="16.497496875" y2="11.112503125" width="0.4064" layer="16"/>
+<wire x1="16.497496875" y1="11.112503125" x2="16.51" y2="11.1" width="0.4064" layer="16"/>
+<wire x1="16.51" y1="10.36" x2="31.229" y2="6.667503125" width="0" layer="19" extent="1-16"/>
 </signal>
 <signal name="N$7">
@@
 <contactref element="T3" pad="B"/>
 <wire x1="16.5075" y1="16.345003125" x2="16.5075" y2="13.970003125" width="0.4064" layer="16"/>
-<wire x1="16.5075" y1="13.970003125" x2="16.51" y2="13.967503125" width="0.4064" layer="16"/>
+<wire x1="16.5075" y1="13.970003125" x2="16.51" y2="13.867503125" width="0.4064" layer="16"/>
 </signal>
 <signal name="N$17">
