File: BRD/gatilhobaixocusto.brd (EAGLE design)
At the start: 41.3 x 21.6 mm, 38 parts, among them IC1 TINY13-20SSU, IC2 LD117AS28TR, Q1 IRL7843, T1 BC817, T2 BC807, T3 BC817

Commit message: Signed-off-by: Jéfferson Pimenta Melo <jefferson.pimenta@hotmail.com>
Parts:
- removed C2: 22uF, rcl:C1210K
- removed C4: 100nF, rcl:C1206K
- removed D2, D3: 4,7v, diode:SOD80C
- removed D4: 4,7V, diode:SOD80C
- removed IC1: TINY13-20SSU, atmel:8S1
- removed IC2: LD117AS28TR, v-reg:SOT223
- removed R11, R5, R6, R7, R8: 10k, resistor:R0805
- removed R3: 9,1k, resistor:R0805
- removed R9: 4k7, resistor:R0805
- removed SJ1, SJ2, SJ3, SJ4: (no value), jumper:SJ
- moved R4 35.1 mm to (2.09, 10.0), turned to 90 degrees
- moved PAD2 33.3 mm to (2.90, 5.50)
- moved C3 21.2 mm to (2.12, 14.6), flipped to the bottom
- moved PAD1 17.7 mm to (14.1, 5.50), turned to 180 degrees
- moved T2 1.10 mm to (6.38, 10.6)
- moved R12 0.90 mm to (5.03, 17.6)
- moved R10 0.30 mm to (7.29, 17.6)
Connections:
- removed net N$10: IC1.1, R7.1
- removed net N$14: BAT+.1, C3.2, D5.C, IC2.3, M+.1, SJ4.1
- removed net N$18: R3.2, SJ4.2
- removed net N$19: R11.1, R8.2, SJ3.2
- removed net N$20: C2.2, C4.2, IC1.8, IC2.4, R10.1, R5.2, R6.2, R7.2, T2.E
- removed net N$6: IC1.5, R1.1, R14.2
- removed net N$8: D3.C, IC1.3, R3.1, R9.1
- removed net N$9: IC1.7, R6.1, SJ1.2
- net N$1: no longer C2.1, C4.1, D2.A, D3.A, D4.A, IC1.4, IC2.1, R11.2, R4.2, R9.2, SJ1.1, SJ2.1
- net N$2: no longer SJ3.1
- net N$5: now also BAT+.1, C3.2, D5.C, M+.1, R10.1, R4.2, T2.E; no longer D4.C, IC1.2, R8.1
- net N$7: now also R1.1, R14.2; no longer D2.C, IC1.6, R5.1, SJ2.2
Routing:
- net N$20: track 29.0 -> 0.00 mm, vias 2 -> 0
- net N$14: track 23.5 -> 0.00 mm, vias 2 -> 0
- net N$5: track 12.5 -> 36.0 mm, vias 0 -> 2
- net N$6: track 11.8 -> 0.00 mm, vias 2 -> 0
- net N$9: track 9.67 -> 0.00 mm, vias 1 -> 0
- net N$8: track 8.22 -> 0.00 mm
- net N$19: track 7.79 -> 0.00 mm
- net N$2: track 26.6 -> 21.7 mm, vias 2 -> 0
- net N$10: track 4.41 -> 0.00 mm
- net N$7: track 13.1 -> 9.19 mm, vias 1 -> 0
- net N$18: track 1.78 -> 0.00 mm
- net N$13: track 6.24 -> 5.14 mm
- net N$11: track 12.0 -> 11.1 mm
- net N$1: vias 4 -> 1
- added copper zone on layer 1, net N$5
- removed copper zone on layer 1, net N$14
Other:
- board size 41.3 x 21.6 mm -> 20.3 x 21.6 mm
- board text added: "J02"
- board text removed: "J01"

Commit message: Signed-off-by: Jéfferson Pimenta Melo <jefferson.pimenta@hotmail.com>
Parts:
- removed D5: SMCJ16A, diode:SMA
- removed R10: 1k, resistor:R0805
- removed R14: 10k, resistor:R0805
- added D2: 15v, diode:SOD80C
- added R3: 1k, resistor:R0805
- added R7: 100R, resistor:R0805
- D1: value 15v -> SMCJ16A; device diode:SOD80C -> diode:SMA
- R2: value 100R -> 10k
- moved D1 14.8 mm to (9.67, 19.2)
- moved R1 14.7 mm to (2.09, 10.0)
- moved R4 9.20 mm to (7.29, 17.6)
- moved T1 8.63 mm to (15.6, 17.4), turned to 0 degrees
- moved T3 8.63 mm to (10.3, 10.6), turned to 180 degrees
- moved R2 8.49 mm to (16.5, 9.40)
- renumbered C3 to C1, PAD1 to PAD4, PAD2 to PAD3, R12 to R5, R13 to R6
Connections:
- net N$1: now also D2.A, R2.1; no longer D1.A, R14.1
- net N$11: now also R4.2, T1.C; no longer R10.2, T3.C
- net N$12: now also R3.2, T1.B; no longer R1.2, T3.B
- net N$13: now also R7.2, T3.C; no longer R2.2, T1.C
- net N$16: now also T3.B; no longer T1.B
- net N$17: now also D2.C, R7.1; no longer D1.C, R2.1
- net N$2: now also D1.A; no longer D5.A
- net N$4: now also R1.1; no longer R4.1
- net N$5: now also D1.C, R1.2, R4.1; no longer D5.C, R10.1, R4.2
- net N$7: now also R2.2, R3.1; no longer R1.1, R14.2
Routing:
- net N$2: track 21.7 -> 23.3 mm

Commit message: Signed-off-by: Jéfferson Pimenta Melo <jefferson.pimenta@hotmail.com>
Parts:
- R3: value 1k -> 10k
- renumbered PAD3 to PAD2, PAD4 to PAD1
Changed lines of the file:
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@@
 <attribute name="VALUE" x="18.57" y="19.467503125" size="0.0254" layer="27" rot="R270"/>
 </element>
-<element name="R3" library="resistor" package="R0805" value="1k" x="16.51" y="12.917503125" smashed="yes" rot="MR90">
+<element name="R3" library="resistor" package="R0805" value="10k" x="16.51" y="12.917503125" smashed="yes" rot="MR90">
 <attribute name="NAME" x="13.97" y="12.917503125" size="1.27" layer="26" rot="MR90"/>
 <attribute name="VALUE" x="13.97" y="12.282503125" size="1.27" layer="28" rot="MR90"/>
@@
 <attribute name="VALUE" x="5.3975" y="8.255003125" size="1.27" layer="27" rot="R90"/>
 </element>
-<element name="PAD4" library="wirepad" package="5-1,8" value="WIREPADSMD5-1,8" x="14.05" y="5.502496875" smashed="yes" rot="MR180">
+<element name="PAD1" library="wirepad" package="5-1,8" value="WIREPADSMD5-1,8" x="14.05" y="5.502496875" smashed="yes" rot="MR180">
 <attribute name="NAME" x="12.1625" y="2.293496875" size="1.27" layer="26" ratio="10" rot="MR180"/>
 <attribute name="VALUE" x="13.95" y="2.702496875" size="0.0254" layer="28" rot="MR180"/>
 </element>
-<element name="PAD3" library="wirepad" package="5-1,8" value="WIREPADSMD5-1,8" x="2.895" y="5.497503125" smashed="yes" rot="MR0">
+<element name="PAD2" library="wirepad" package="5-1,8" value="WIREPADSMD5-1,8" x="2.895" y="5.497503125" smashed="yes" rot="MR0">
 <attribute name="NAME" x="5.635" y="1.006503125" size="1.27" layer="26" ratio="10" rot="MR0"/>
 <attribute name="VALUE" x="2.995" y="8.297503125" size="0.0254" layer="28" rot="MR0"/>
@@
 </signal>
 <signal name="N$7">
-<contactref element="PAD4" pad="1"/>
+<contactref element="PAD1" pad="1"/>
 <contactref element="R3" pad="1"/>
 <contactref element="R2" pad="2"/>
@@
 <signal name="N$4">
 <contactref element="R1" pad="1"/>
-<contactref element="PAD3" pad="1"/>
+<contactref element="PAD2" pad="1"/>
 <wire x1="2.895" y1="5.497503125" x2="2.895" y2="8.105" width="0.4064" layer="16"/>
 <wire x1="2.895" y1="8.105" x2="2.1" y2="8.9" width="0.4064" layer="16"/>
