File: BRD/gatilhobaixocusto.sch (EAGLE design)
At the start: 20 parts, among them Q1 IRL7843, T1 BC817, T2 BC807, T3 BC817

Commit message: Signed-off-by: Jéfferson Pimenta Melo <jefferson.pimenta@hotmail.com>
Parts:
- removed D5: SMCJ16A, diode:MBRA340T3
- removed R10: 1k, resistor:R-EU_R0805
- removed R14: 10k, resistor:R-EU_R0805
- added D2: 15v, diode:ZENER-DIODESOD80C
- added R3: 1k, resistor:R-EU_R0805
- added R7: 100R, resistor:R-EU_R0805
- D1: value 15v -> SMCJ16A; device diode:ZENER-DIODESOD80C -> diode:MBRA340T3
- R2: value 100R -> 10k
- renumbered C3 to C1, PAD1 to PAD4, PAD2 to PAD3, R12 to R5, R13 to R6
Connections:
- net N$1: now also D2.A, R2.1; no longer D1.A, R14.1
- net N$11: now also R4.2, T1.C; no longer R10.2, T3.C
- net N$12: now also R3.2, T1.B; no longer R1.2, T3.B
- net N$13: now also R7.2, T3.C; no longer R2.2, T1.C
- net N$16: now also T3.B; no longer T1.B
- net N$17: now also D2.C, R7.1; no longer D1.C, R2.1
- net N$2: now also D1.A; no longer D5.A
- net N$4: now also R1.1; no longer R4.1
- net N$5: now also D1.C, R1.2, R4.1; no longer D5.C, R10.1, R4.2
- net N$7: now also R2.2, R3.1; no longer R1.1, R14.2
Other:
- moved on the sheet: R1, R2, R4, T1, T3

Commit message: Signed-off-by: Jéfferson Pimenta Melo <jefferson.pimenta@hotmail.com>
Parts:
- R3: value 1k -> 10k
- renumbered PAD3 to PAD2, PAD4 to PAD1
Changed lines of the file:
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@@
 <part name="M-" library="wirepad" deviceset="WIREPAD" device="SMD5-2,5"/>
 <part name="BAT-" library="wirepad" deviceset="WIREPAD" device="SMD5-2,5"/>
-<part name="R3" library="resistor" deviceset="R-EU_" device="R0805" value="1k"/>
+<part name="R3" library="resistor" deviceset="R-EU_" device="R0805" value="10k"/>
 <part name="D2" library="diode" deviceset="ZENER-DIODE" device="SOD80C" value="15v"/>
 <part name="T3" library="transistor-neu-to92" deviceset="*-NPN-" device="SOT23-BEC" technology="MMBT3904LT1" value="BC817"/>
@@
 <part name="C1" library="rcl" deviceset="C-EU" device="C0805K" value="100nF"/>
 <part name="Q1" library="transistor-fet" deviceset="FDD4141" device="TO252" value="IRL7843"/>
-<part name="PAD4" library="wirepad" deviceset="WIREPAD" device="SMD5-1,8"/>
-<part name="PAD3" library="wirepad" deviceset="WIREPAD" device="SMD5-1,8"/>
+<part name="PAD1" library="wirepad" deviceset="WIREPAD" device="SMD5-1,8"/>
+<part name="PAD2" library="wirepad" deviceset="WIREPAD" device="SMD5-1,8"/>
 <part name="D1" library="diode" deviceset="MBRA340T3" device="" value="SMCJ16A"/>
 <part name="R1" library="resistor" deviceset="R-EU_" device="R0805" value="1k"/>
@@
 <instance part="C1" gate="G$1" x="60.96" y="66.04" rot="R180"/>
 <instance part="Q1" gate="G$1" x="226.06" y="60.96" rot="MR180"/>
-<instance part="PAD4" gate="G$1" x="101.6" y="58.42"/>
-<instance part="PAD3" gate="G$1" x="96.52" y="58.42" rot="R180"/>
+<instance part="PAD1" gate="G$1" x="101.6" y="58.42"/>
+<instance part="PAD2" gate="G$1" x="96.52" y="58.42" rot="R180"/>
 <instance part="D1" gate="G$1" x="205.74" y="83.82" rot="R90"/>
 <instance part="R1" gate="G$1" x="86.36" y="58.42" rot="R180"/>
@@
 <net name="N$7" class="0">
 <segment>
-<pinref part="PAD4" gate="G$1" pin="P"/>
+<pinref part="PAD1" gate="G$1" pin="P"/>
 <pinref part="R3" gate="G$1" pin="1"/>
 <wire x1="129.54" y1="58.42" x2="127" y2="58.42" width="0.1524" layer="91"/>
@@
 <segment>
 <pinref part="R1" gate="G$1" pin="1"/>
-<pinref part="PAD3" gate="G$1" pin="P"/>
+<pinref part="PAD2" gate="G$1" pin="P"/>
 <wire x1="93.98" y1="58.42" x2="91.44" y2="58.42" width="0.1524" layer="91"/>
 </segment>
